Commit message: upd

File: src/hexa_description/urdf/hexa.urdf (robot description, URDF)
Before this commit: robot hexo, 25 links, 24 joints
Links:
- added link lidar_link, mass 0.000010; visual mesh filename=package://hexa_description/meshes/stl/hexo_base_v1.003.stl scale=1.000000 1.000000 1.000000
- added link rgbd_link, mass 0.000010; visual mesh filename=package://hexa_description/meshes/stl/hexo_base_v1.stl scale=1.000000 1.000000 1.000000
- link base_link: mass None -> 0.000010; geometry visual mesh filename=package://hexa_description/meshes/stl/hexo_base_v1.001.stl scale=1.000000 1.000000 1.000000
- link leg1_link1: mass None -> 0.000010; geometry visual mesh filename=package://hexa_description/meshes/stl/hexo_full.007.stl scale=1.000000 1.000000 1.000000
- link leg1_link2: mass None -> 0.000010; geometry visual mesh filename=package://hexa_description/meshes/stl/hexo_full.008.stl scale=1.000000 1.000000 1.000000
- link leg1_link3: mass None -> 0.000010; geometry visual mesh filename=package://hexa_description/meshes/stl/hexo_full.009.stl scale=1.000000 1.000000 1.000000
- link leg1_link4: mass None -> 0.000010
- link leg2_link1: mass None -> 0.000010; geometry visual mesh filename=package://hexa_description/meshes/stl/hexo_full.004.stl scale=1.000000 1.000000 1.000000
- link leg2_link2: mass None -> 0.000010; geometry visual mesh filename=package://hexa_description/meshes/stl/hexo_full.005.stl scale=1.000000 1.000000 1.000000
- link leg2_link3: mass None -> 0.000010; geometry visual mesh filename=package://hexa_description/meshes/stl/hexo_full.006.stl scale=1.000000 1.000000 1.000000
- link leg2_link4: mass None -> 0.000010
- link leg3_link1: mass None -> 0.000010; geometry visual mesh filename=package://hexa_description/meshes/stl/hexo_full.019.stl scale=1.000000 1.000000 1.000000
- link leg3_link2: mass None -> 0.000010; geometry visual mesh filename=package://hexa_description/meshes/stl/hexo_full.020.stl scale=1.000000 1.000000 1.000000
- link leg3_link3: mass None -> 0.000010; geometry visual mesh filename=package://hexa_description/meshes/stl/hexo_full.021.stl scale=1.000000 1.000000 1.000000
- link leg3_link4: mass None -> 0.000010
- link leg4_link1: mass None -> 0.000010; geometry visual mesh filename=package://hexa_description/meshes/stl/hexo_full.016.stl scale=1.000000 1.000000 1.000000
- link leg4_link2: mass None -> 0.000010; geometry visual mesh filename=package://hexa_description/meshes/stl/hexo_full.017.stl scale=1.000000 1.000000 1.000000
- link leg4_link3: mass None -> 0.000010; geometry visual mesh filename=package://hexa_description/meshes/stl/hexo_full.022.stl scale=1.000000 1.000000 1.000000
- link leg4_link4: mass None -> 0.000010
- link leg5_link1: mass None -> 0.000010; geometry visual mesh filename=package://hexa_description/meshes/stl/hexo_full.013.stl scale=1.000000 1.000000 1.000000
- link leg5_link2: mass None -> 0.000010; geometry visual mesh filename=package://hexa_description/meshes/stl/hexo_full.014.stl scale=1.000000 1.000000 1.000000
- link leg5_link3: mass None -> 0.000010; geometry visual mesh filename=package://hexa_description/meshes/stl/hexo_full.015.stl scale=1.000000 1.000000 1.000000
- link leg5_link4: mass None -> 0.000010
- link leg6_link1: mass None -> 0.000010; geometry visual mesh filename=package://hexa_description/meshes/stl/hexo_full.010.stl scale=1.000000 1.000000 1.000000
- link leg6_link2: mass None -> 0.000010; geometry visual mesh filename=package://hexa_description/meshes/stl/hexo_full.011.stl scale=1.000000 1.000000 1.000000
- link leg6_link3: mass None -> 0.000010; geometry visual mesh filename=package://hexa_description/meshes/stl/hexo_full.012.stl scale=1.000000 1.000000 1.000000
- link leg6_link4: mass None -> 0.000010
Joints:
- added joint lidar_joint: type fixed, parent base_link, child lidar_link, origin xyz=-0.000038 -0.000818 0.108350 rpy=0.000000 0.000000 0.000000
- added joint rgbd_joint: type fixed, parent base_link, child rgbd_link, origin xyz=0.080951 0.000000 0.084500 rpy=0.000000 0.000000 0.000000
- joint leg1_link1_joint: origin xyz=0.075777 -0.043750 -0.000000 rpy=0.000000 0.000000 -0.523598 -> xyz=0.077942 -0.045000 0.024150 rpy=0.000000 0.000000 -0.523598
- joint leg1_link2_joint: origin xyz=0.080000 -0.000000 0.000000 rpy=0.000000 0.000000 -0.000000 -> xyz=0.070590 -0.000900 0.000072 rpy=0.000000 0.000000 -0.000000
- joint leg1_link3_joint: origin xyz=0.080000 -0.000000 -0.000000 rpy=0.000000 0.000000 0.000000 -> xyz=0.079450 -0.000900 -0.000072 rpy=0.000000 0.000000 0.000000
- joint leg1_link4_joint: origin xyz=0.034000 -0.000000 -0.111000 rpy=0.000000 0.000000 0.000000 -> xyz=0.033000 -0.000000 -0.100000 rpy=0.000000 0.000000 0.000000
- joint leg2_link1_joint: origin xyz=0.000000 -0.087500 -0.000000 rpy=0.000000 0.000000 -1.570796 -> xyz=0.000000 -0.089999 0.024150 rpy=0.000000 0.000000 -1.570796
- joint leg2_link2_joint: origin xyz=0.080000 -0.000000 0.000000 rpy=0.000000 0.000000 0.000000 -> xyz=0.070590 -0.000900 0.000072 rpy=0.000000 0.000000 0.000000
- joint leg2_link3_joint: origin xyz=0.080000 -0.000000 0.000000 rpy=0.000000 0.000000 0.000000 -> xyz=0.079450 -0.000900 -0.000072 rpy=0.000000 0.000000 0.000000
- joint leg2_link4_joint: origin xyz=0.034000 -0.000000 -0.111000 rpy=0.000000 0.000000 -0.000000 -> xyz=0.033000 -0.000000 -0.100000 rpy=0.000000 0.000000 -0.000000
- joint leg3_link1_joint: origin xyz=-0.075777 -0.043750 -0.000000 rpy=0.000000 0.000000 -2.617994 -> xyz=-0.077942 -0.045000 0.024150 rpy=0.000000 0.000000 -2.617994
- joint leg3_link2_joint: origin xyz=0.080000 -0.000000 0.000000 rpy=0.000000 0.000000 0.000000 -> xyz=0.070590 -0.000900 0.000072 rpy=0.000000 0.000000 0.000000
- joint leg3_link3_joint: origin xyz=0.080000 -0.000000 0.000000 rpy=0.000000 0.000000 0.000000 -> xyz=0.079450 -0.000900 -0.000072 rpy=0.000000 0.000000 0.000000
- joint leg3_link4_joint: origin xyz=0.034000 -0.000000 -0.111000 rpy=0.000000 0.000000 0.000000 -> xyz=0.033000 -0.000000 -0.100000 rpy=0.000000 0.000000 0.000000
- joint leg4_link1_joint: origin xyz=-0.075777 0.043750 -0.000000 rpy=0.000000 0.000000 2.617994 -> xyz=-0.077942 0.045000 0.024150 rpy=0.000000 0.000000 2.617994
- joint leg4_link2_joint: origin xyz=0.080000 -0.000000 0.000000 rpy=0.000000 0.000000 -0.000000 -> xyz=0.070590 -0.000900 0.000072 rpy=0.000000 0.000000 -0.000000
- joint leg4_link3_joint: origin xyz=0.080000 0.000000 0.000000 rpy=0.000000 0.000000 -0.000000 -> xyz=0.079450 -0.000900 -0.000072 rpy=0.000000 0.000000 -0.000000
- joint leg4_link4_joint: origin xyz=0.034000 0.000000 -0.111000 rpy=0.000000 0.000000 -0.000000 -> xyz=0.033000 0.000000 -0.100000 rpy=0.000000 0.000000 -0.000000
- joint leg5_link1_joint: origin xyz=-0.000000 0.087500 -0.000000 rpy=0.000000 0.000000 1.570796 -> xyz=-0.000000 0.089999 0.024150 rpy=0.000000 0.000000 1.570796
- joint leg5_link2_joint: origin xyz=0.080000 -0.000000 0.000000 rpy=0.000000 0.000000 -0.000000 -> xyz=0.070590 -0.000900 0.000072 rpy=0.000000 0.000000 -0.000000
- joint leg5_link3_joint: origin xyz=0.080000 -0.000000 -0.000000 rpy=0.000000 0.000000 0.000000 -> xyz=0.079450 -0.000900 -0.000072 rpy=0.000000 0.000000 0.000000
- joint leg5_link4_joint: origin xyz=0.034000 -0.000000 -0.111000 rpy=0.000000 0.000000 0.000000 -> xyz=0.033000 -0.000000 -0.100000 rpy=0.000000 0.000000 0.000000
- joint leg6_link1_joint: origin xyz=0.075777 0.043750 -0.000000 rpy=0.000000 0.000000 0.523599 -> xyz=0.077942 0.045000 0.024150 rpy=0.000000 0.000000 0.523599
- joint leg6_link2_joint: origin xyz=0.080000 -0.000000 0.000000 rpy=0.000000 0.000000 0.000000 -> xyz=0.070590 -0.000900 0.000072 rpy=0.000000 0.000000 0.000000
- joint leg6_link3_joint: origin xyz=0.080000 -0.000000 0.000000 rpy=0.000000 0.000000 -0.000000 -> xyz=0.079450 -0.000900 -0.000072 rpy=0.000000 0.000000 -0.000000
- joint leg6_link4_joint: origin xyz=0.034000 -0.000000 -0.111000 rpy=0.000000 0.000000 -0.000000 -> xyz=0.033000 -0.000000 -0.100000 rpy=0.000000 0.000000 -0.000000

File: src/hexa_description/urdf/hexa_old.urdf (robot description, URDF)
Before this commit: robot hexa, 25 links, 24 joints
Links:
- link base_link: mass 0.000010 -> None
- link leg1_link1: mass 0.000010 -> None
- link leg1_link2: mass 0.000010 -> None
- link leg1_link3: mass 0.000010 -> None
- link leg1_link4: mass 0.000010 -> None
- link leg2_link1: mass 0.000010 -> None
- link leg2_link2: mass 0.000010 -> None
- link leg2_link3: mass 0.000010 -> None
- link leg2_link4: mass 0.000010 -> None
- link leg3_link1: mass 0.000010 -> None
- link leg3_link2: mass 0.000010 -> None
- link leg3_link3: mass 0.000010 -> None
- link leg3_link4: mass 0.000010 -> None
- link leg4_link1: mass 0.000010 -> None
- link leg4_link2: mass 0.000010 -> None
- link leg4_link3: mass 0.000010 -> None
- link leg4_link4: mass 0.000010 -> None
- link leg5_link1: mass 0.000010 -> None
- link leg5_link2: mass 0.000010 -> None
- link leg5_link3: mass 0.000010 -> None
- link leg5_link4: mass 0.000010 -> None
- link leg6_link1: mass 0.000010 -> None
- link leg6_link2: mass 0.000010 -> None
- link leg6_link3: mass 0.000010 -> None
- link leg6_link4: mass 0.000010 -> None
Joints:
- joint leg1_link2_joint: axis 0.000000 1.000000 0.000000 -> 0.000000 -1.000000 0.000000; limit lower=-2.000000 upper=2.000000 effort=1.960000 velocity=5.220000 -> lower=-2.000000 upper=2.000000 effort=1.960000 velocity=0.000000
- joint leg1_link3_joint: axis 0.000000 1.000000 0.000000 -> 0.000000 -1.000000 0.000000; limit lower=-2.000000 upper=2.000000 effort=1.960000 velocity=5.220000 -> lower=-2.000000 upper=2.000000 effort=1.960000 velocity=0.000000
- joint leg2_link2_joint: axis 0.000000 1.000000 0.000000 -> 0.000000 -1.000000 0.000000; limit lower=-2.000000 upper=2.000000 effort=1.960000 velocity=5.220000 -> lower=-2.000000 upper=2.000000 effort=1.960000 velocity=0.000000
- joint leg2_link3_joint: axis 0.000000 1.000000 0.000000 -> 0.000000 -1.000000 0.000000; limit lower=-2.000000 upper=2.000000 effort=1.960000 velocity=5.220000 -> lower=-2.000000 upper=2.000000 effort=1.960000 velocity=0.000000
- joint leg3_link2_joint: axis 0.000000 1.000000 0.000000 -> 0.000000 -1.000000 0.000000; limit lower=-2.000000 upper=2.000000 effort=1.960000 velocity=5.220000 -> lower=-2.000000 upper=2.000000 effort=1.960000 velocity=0.000000
- joint leg3_link3_joint: axis 0.000000 1.000000 0.000000 -> 0.000000 -1.000000 0.000000; limit lower=-2.000000 upper=2.000000 effort=1.960000 velocity=5.220000 -> lower=-2.000000 upper=2.000000 effort=1.960000 velocity=0.000000
- joint leg4_link2_joint: axis 0.000000 1.000000 0.000000 -> 0.000000 -1.000000 0.000000; limit lower=-2.000000 upper=2.000000 effort=1.960000 velocity=5.220000 -> lower=-2.000000 upper=2.000000 effort=1.960000 velocity=0.000000
- joint leg4_link3_joint: axis 0.000000 1.000000 0.000000 -> 0.000000 -1.000000 0.000000; limit lower=-2.000000 upper=2.000000 effort=1.960000 velocity=5.220000 -> lower=-2.000000 upper=2.000000 effort=1.960000 velocity=0.000000
- joint leg5_link2_joint: axis 0.000000 1.000000 0.000000 -> 0.000000 -1.000000 0.000000; limit lower=-2.000000 upper=2.000000 effort=1.960000 velocity=5.220000 -> lower=-2.000000 upper=2.000000 effort=1.960000 velocity=0.000000
- joint leg5_link3_joint: axis 0.000000 1.000000 0.000000 -> 0.000000 -1.000000 0.000000; limit lower=-2.000000 upper=2.000000 effort=1.960000 velocity=5.220000 -> lower=-2.000000 upper=2.000000 effort=1.960000 velocity=0.000000; origin xyz=0.080000 -0.000000 0.000000 rpy=0.000000 0.000000 0.000000 -> xyz=0.080000 -0.000000 -0.000000 rpy=0.000000 0.000000 0.000000
- joint leg6_link2_joint: axis 0.000000 1.000000 0.000000 -> 0.000000 -1.000000 0.000000; limit lower=-2.000000 upper=2.000000 effort=1.960000 velocity=5.220000 -> lower=-2.000000 upper=2.000000 effort=1.960000 velocity=0.000000
- joint leg6_link3_joint: axis 0.000000 1.000000 0.000000 -> 0.000000 -1.000000 0.000000; limit lower=-2.000000 upper=2.000000 effort=1.960000 velocity=5.220000 -> lower=-2.000000 upper=2.000000 effort=1.960000 velocity=0.000000

Commit message: upd

File: src/hexa_description/urdf/hexa.urdf (robot description, URDF)
Before this commit: robot hexo, 27 links, 26 joints
Links:
- removed link lidar_link
- added link base_laser, mass 0.000010; visual mesh filename=package://hexa_description/meshes/stl/hexo_base_v1.003.stl scale=1.000000 1.000000 1.000000
Joints:
- joint lidar_joint: child lidar_link -> base_laser
